Commit message: init

File: src/xarm/urdf/arm_only_xarm.urdf.xacro (robot description, xacro)
@@ -42,19 +42,17 @@
       <xacro:controlled_joint joint_name="arm_5_joint" />
       <xacro:controlled_joint joint_name="arm_6_joint" />
-      <xacro:controlled_joint joint_name="gripper_1_joint" />
-      <joint name="gripper_2_joint">
-        <param name="mimic">gripper_1_joint</param>
-        <param name="multiplier">1.0</param>
-        <xacro:unless value="${hardware_type == 'gz'}">
-          <command_interface name="position" />
-          <state_interface name="position" />
-          <state_interface name="velocity" />
-        </xacro:unless>
-      </joint>
+       <xacro:controlled_joint joint_name="gripper_1_joint" />
+       <xacro:controlled_joint joint_name="gripper_2_joint" />
     </ros2_control>
   </xacro:macro>
-  <xacro:xarm
-    include_world_joint="$(arg include_world_joint)"
-    base_height="$(arg base_height)" />
+  <xacro:xarm gripper_mimic="false" gripper_lower_limit="-0.05" />
+  <xacro:if value="$(arg include_world_joint)">
+    <link name="world" />
+    <joint name="world_joint" type="fixed">
+      <parent link="world" />
+      <child link="base_link" />
+      <origin xyz="0 0 $(arg base_height)" rpy="0 0 0" />
+    </joint>
+  </xacro:if>
   <xacro:if value="$(arg use_ros2_control)">
     <xacro:arm_only_ros2_control
@@ -63,4 +61,10 @@
       initial_positions_file="$(arg initial_positions_file)" />
   </xacro:if>
+  <gazebo reference="gripper_1_link">
+    <gravity>false</gravity>
+  </gazebo>
+  <gazebo reference="gripper_2_link">
+    <gravity>false</gravity>
+  </gazebo>
   <xacro:if value="${selected_hardware_type == 'gz'}">
     <gazebo>

File: src/xarm_description/urdf/arm.urdf.xacro (robot description, xacro)
@@ -3,5 +3,5 @@
 <xacro:property name="arm_friction"       value="1.0" />
 <xacro:property name="arm_damping"        value="1.0" />
-<xacro:macro name="xarm" >
+<xacro:macro name="xarm" params="gripper_mimic:=true gripper_lower_limit:=0.0">
   <!-- link name="world" / -->
   <!--joint name="virtual_joint" type="fixed">
@@ -413,5 +413,5 @@
       xyz="0 0 1" />
     <limit
-      lower="0"
+       lower="${gripper_lower_limit}"
       upper="0.698"
       effort="100"
@@ -470,12 +470,14 @@
       xyz="0 0 1" />
     <limit
-      lower="0"
+       lower="${gripper_lower_limit}"
       upper="0.698"
       effort="100"
       velocity="0.35" />
     <dynamics friction="${arm_friction}" damping="${arm_damping}"/>
-    <mimic joint="gripper_1_joint" >
-      <multiplier>1</multiplier>
-    </mimic>
+    <xacro:if value="${gripper_mimic}">
+      <mimic joint="gripper_1_joint">
+        <multiplier>1</multiplier>
+      </mimic>
+    </xacro:if>
   </joint>
   <link

File: src/xarm_description/urdf/xarm.ros2_control.xacro (robot description, xacro)
@@ -3,5 +3,5 @@
   <xacro:macro
     name="xarm_ros2_control"
-    params="name hardware_type initial_positions_file">
+    params="name hardware_type initial_positions_file gripper_mimic:=true">
     <xacro:property
       name="initial_positions"
@@ -35,4 +35,13 @@
       <xacro:controlled_joint joint_name="arm_6_joint" />
       <xacro:controlled_joint joint_name="gripper_1_joint" />
+      <xacro:if value="${gripper_mimic}">
+        <joint name="gripper_2_joint">
+          <param name="mimic">gripper_1_joint</param>
+          <param name="multiplier">1.0</param>
+        </joint>
+      </xacro:if>
+      <xacro:unless value="${gripper_mimic}">
+        <xacro:controlled_joint joint_name="gripper_2_joint" />
+      </xacro:unless>
     </ros2_control>
   </xacro:macro>

File: src/xarm_description/urdf/xarm.urdf.xacro (robot description, xacro)
@@ -12,10 +12,11 @@
   <xacro:include filename="$(find xarm_description)/urdf/arm.urdf.xacro" />
   <xacro:include filename="$(find xarm_description)/urdf/xarm.ros2_control.xacro" />
-  <xacro:xarm />
+  <xacro:xarm gripper_mimic="true" />
   <xacro:if value="$(arg use_ros2_control)">
     <xacro:xarm_ros2_control
       name="XBotArmSystem"
       hardware_type="${selected_hardware_type}"
-      initial_positions_file="$(arg initial_positions_file)" />
+      initial_positions_file="$(arg initial_positions_file)"
+      gripper_mimic="true" />
   </xacro:if>
   <xacro:if value="${selected_hardware_type == 'gz'}">
